Commit message: Add a controller package

File: six_dof_cam_description/urdf/camera/camera.gazebo.xacro (robot description, xacro)
@@ -4,6 +4,4 @@
 		<gazebo reference="camera_link">
 			<!-- <selfCollide>true</selfCollide> -->
-			<!-- <mu1 value="0.05" /> -->
-			<!-- <mu2 value="0.05" /> -->
 			<mu1>0.05</mu1>
 			<mu2>0.05</mu2>

File: six_dof_cam_description/urdf/camera/camera.xacro (robot description, xacro)
@@ -6,5 +6,5 @@
 	<xacro:macro name="camera" params="parent *joint_origin">
 		<joint name="camera_joint" type="fixed">
-			<insert_block name="joint_origin"/>
+			<xacro:insert_block name="joint_origin"/>
 			<parent link="${parent}"/>
 			<child link="camera_link"/>

File: six_dof_cam_description/urdf/linear_actuator/linear_actuator.gazebo.xacro (robot description, xacro)
@@ -2,8 +2,6 @@
 <robot xmlns:xacro="http://ros.org/wiki/xacro">
 	<xacro:macro name="linear_actuator_gazebo" params="prefix">
-		<gazebo reference="${prefix}_linear_actuator">
+		<gazebo reference="${prefix}_linear_actuator_link">
 			<!-- <selfCollide>true</selfCollide> -->
-			<!-- <mu1 value="0.05" /> -->
-			<!-- <mu2 value="0.05" /> -->
 			<mu1>0.05</mu1>
 			<mu2>0.05</mu2>

File: six_dof_cam_description/urdf/linear_actuator/linear_actuator.xacro (robot description, xacro)
@@ -2,10 +2,11 @@
 <robot xmlns:xacro="http://ros.org/wiki/xacro">
 	<xacro:include filename="$(find six_dof_cam_description)/urdf/linear_actuator/linear_actuator.gazebo.xacro"/>
+	<xacro:include filename="$(find six_dof_cam_description)/urdf/linear_actuator/linear_actuator.transmission.xacro"/>
 	<xacro:property name="M_PI" value="3.1415926535897931" />
 	<xacro:property name="velocity_scale_factor" value="1.0"/>
 	<xacro:macro name="linear_actuator" params="prefix parent *joint_origin *joint_axis">
 		<joint name="${prefix}_linear_actuator_joint" type="prismatic">
-			<insert_block name="joint_origin"/>
-			<insert_block name="joint_axis"/>
+			<xacro:insert_block name="joint_origin"/>
+			<xacro:insert_block name="joint_axis"/>
 			<parent link="${parent}"/>
 			<child link="${prefix}_linear_actuator_link"/>

File: six_dof_cam_description/urdf/rotary_actuator/rotary_actuator.gazebo.xacro (robot description, xacro)
@@ -2,8 +2,6 @@
 <robot xmlns:xacro="http://ros.org/wiki/xacro">
 	<xacro:macro name="rotary_actuator_gazebo" params="prefix">
-		<gazebo reference="${prefix}_rotary_actuator">
+		<gazebo reference="${prefix}_rotary_actuator_link">
 			<!-- <selfCollide>true</selfCollide> -->
-			<!-- <mu1 value="0.05" /> -->
-			<!-- <mu2 value="0.05" /> -->
 			<mu1>0.05</mu1>
 			<mu2>0.05</mu2>

File: six_dof_cam_description/urdf/rotary_actuator/rotary_actuator.xacro (robot description, xacro)
@@ -2,10 +2,11 @@
 <robot xmlns:xacro="http://ros.org/wiki/xacro">
 	<xacro:include filename="$(find six_dof_cam_description)/urdf/rotary_actuator/rotary_actuator.gazebo.xacro"/>
+	<xacro:include filename="$(find six_dof_cam_description)/urdf/rotary_actuator/rotary_actuator.transmission.xacro"/>
 	<xacro:property name="M_PI" value="3.1415926535897931" />
 	<xacro:property name="velocity_scale_factor" value="1.0"/>
 	<xacro:macro name="rotary_actuator" params="prefix parent *joint_origin *joint_axis">
 		<joint name="${prefix}_rotary_actuator_joint" type="revolute">
-			<insert_block name="joint_origin"/>
-			<insert_block name="joint_axis"/>
+			<xacro:insert_block name="joint_origin"/>
+			<xacro:insert_block name="joint_axis"/>
 			<parent link="${parent}"/>
 			<child link="${prefix}_rotary_actuator_link"/>

File: six_dof_cam_description/urdf/six_dof_cam.urdf (robot description, URDF)
Before this commit: robot six_dof_cam, 8 links, 7 joints
Links:
- removed link map
- added link world
Joints:
- joint x_linear_actuator_joint: origin xyz=0 0 0 rpy=0 0 0 -> xyz=0 0 1 rpy=0 0 0; parent map -> world

File: six_dof_cam_description/urdf/six_dof_cam.xacro (robot description, xacro)
@@ -6,7 +6,7 @@
 	<xacro:include filename="$(find six_dof_cam_description)/urdf/rotary_actuator/rotary_actuator.xacro"/>
 <!-- =============== Link & Joint =============== -->
-	<link name="map"/>
-	<xacro:linear_actuator prefix="x" parent="map">
-		<origin xyz="0 0 0" rpy="0 0 0"/>
+	<link name="world"/>
+	<xacro:linear_actuator prefix="x" parent="world">
+		<origin xyz="0 0 1" rpy="0 0 0"/>
 		<axis xyz="1 0 0"/>
 	</xacro:linear_actuator>
@@ -35,24 +35,24 @@
 	</xacro:camera>
 <!-- ===============  Transmission =============== -->
-<!-- PositionJointInterface: requires position -->
-<!-- <xacro:wheel_trans prefix="right" interface="PositionJointInterface"/> -->
-<!-- <xacro:wheel_trans prefix="left" interface="PositionJointInterface"/>  -->
-<!-- VelocityJointInterface: requires position, velocity -->
-<!-- for DiffDriveController -->
-<!--<xacro:wheel_trans prefix="right" interface="hardware_interface/VelocityJointInterface"/>-->
-<!--<xacro:wheel_trans prefix="left" interface="hardware_interface/VelocityJointInterface"/>-->
-<!-- EffortJointInterface: requires position, velocity, effort -->
-<!-- <xacro:wheel_trans prefix="right" interface="EffortJointInterface"/> -->
-<!-- <xacro:wheel_trans prefix="left" interface="EffortJointInterface"/>  -->
+<xacro:linear_actuator_trans prefix="x" interface="hardware_interface/PositionJointInterface"/>
+<xacro:linear_actuator_trans prefix="y" interface="hardware_interface/PositionJointInterface"/>
+<xacro:linear_actuator_trans prefix="z" interface="hardware_interface/PositionJointInterface"/>
+<xacro:rotary_actuator_trans prefix="x" interface="hardware_interface/PositionJointInterface"/>
+<xacro:rotary_actuator_trans prefix="y" interface="hardware_interface/PositionJointInterface"/>
+<xacro:rotary_actuator_trans prefix="z" interface="hardware_interface/PositionJointInterface"/>
 <!-- =============== Gazebo =============== -->
-<!--<gazebo>-->
-<!--<plugin name="gazebo_ros_control" filename="libgazebo_ros_control.so">-->
-<!--<robotNamespace>raspimouse_on_gazebo</robotNamespace>-->
-<!--</plugin>-->
-<!--</gazebo>-->
-<!-- Base -->
-<!--<xacro:base_gazebo/>-->
-<!-- Wheel -->
-<!--<xacro:wheel_gazebo prefix="right"/>-->
-<!--<xacro:wheel_gazebo prefix="left"/>-->
+<gazebo>
+	<plugin name="gazebo_ros_control" filename="libgazebo_ros_control.so">
+		<robotNamespace>six_dof_cam</robotNamespace>
+	</plugin>
+</gazebo>
+<!-- camera -->
+<xacro:camera_gazebo/>
+<!-- actuators -->
+<xacro:rotary_actuator_gazebo prefix="x"/>
+<xacro:rotary_actuator_gazebo prefix="y"/>
+<xacro:rotary_actuator_gazebo prefix="z"/>
+<xacro:linear_actuator_gazebo prefix="x"/>
+<xacro:linear_actuator_gazebo prefix="y"/>
+<xacro:linear_actuator_gazebo prefix="z"/>
 </robot>
