Commit message: display box

File: six_dof_cam_description/urdf/camera/camera.xacro (robot description, xacro)
@@ -22,5 +22,5 @@
 			</collision>
 			<inertial>
-				<origin xyz="0 0 0"/>
+				<origin xyz="0 0 0" rpy="0 0 0"/>
 				<mass value="1.0"/>
 				<inertia ixx="1.0" ixy="0.0" iyy="1.0" ixz="0.0" iyz="0.0" izz="1.0"/>

File: six_dof_cam_description/urdf/six_dof_cam.xacro (robot description, xacro)
@@ -25,9 +25,9 @@
 <!-- <xacro:wheel_trans prefix="left" interface="EffortJointInterface"/>  -->
 <!-- =============== Gazebo =============== -->
-<!--<gazebo>
-<plugin name="gazebo_ros_control" filename="libgazebo_ros_control.so">
-<robotNamespace>raspimouse_on_gazebo</robotNamespace>
-</plugin>
-</gazebo>-->
+<!--<gazebo>-->
+<!--<plugin name="gazebo_ros_control" filename="libgazebo_ros_control.so">-->
+<!--<robotNamespace>raspimouse_on_gazebo</robotNamespace>-->
+<!--</plugin>-->
+<!--</gazebo>-->
 <!-- Base -->
 <!--<xacro:base_gazebo/>-->
@@ -35,4 +35,3 @@
 <!--<xacro:wheel_gazebo prefix="right"/>-->
 <!--<xacro:wheel_gazebo prefix="left"/>-->
-	<six_dof_cam/>
 </robot>

Commit message: add gazebo files

File: six_dof_cam_description/urdf/camera/camera.xacro (robot description, xacro)
@@ -1,5 +1,5 @@
 <?xml version="1.0"?>
 <robot xmlns:xacro="http://ros.org/wiki/xacro">
-	<!--<xacro:include filename="$(find raspimouse_description)/urdf/body/body.gazebo.xacro"/>-->
+	<xacro:include filename="$(find six_dof_cam_description)/urdf/camera/camera.gazebo.xacro"/>
 	<!--<xacro:property name="M_PI" value="3.1415926535897931" />-->
 	<!--<xacro:property name="velocity_scale_factor" value="1.0"/>-->

File: six_dof_cam_description/urdf/rotary_actuator/rotary_actuator.xacro (robot description, xacro)
@@ -1,16 +1,16 @@
 <?xml version="1.0"?>
 <robot xmlns:xacro="http://ros.org/wiki/xacro">
-	<xacro:include filename="$(find six_dof_cam_description)/urdf/linear_actuator/linear_actuator.gazebo.xacro"/>
+	<xacro:include filename="$(find six_dof_cam_description)/urdf/rotary_actuator/rotary_actuator.gazebo.xacro"/>
 	<xacro:property name="M_PI" value="3.1415926535897931" />
 	<xacro:property name="velocity_scale_factor" value="1.0"/>
-	<xacro:macro name="linear_actuator" params="prefix parent *joint_origin *joint_axis">
-		<joint name="${prefix}_linear_actuator_joint" type="prismatic">
+	<xacro:macro name="rotary_actuator" params="prefix parent *joint_origin *joint_axis">
+		<joint name="${prefix}_rotary_actuator_joint" type="revolute">
 			<insert_block name="joint_origin"/>
 			<insert_block name="joint_axis"/>
 			<parent link="${parent}"/>
-			<child link="${prefix}_linear_actuator_link"/>
-			<limit lower="-1" upper="1" effort="0.5" velocity="5.0"/>
+			<child link="${prefix}_rotary_actuator_link"/>
+			<limit lower="-3.14" upper="3.14" effort="0.5" velocity="5.0"/>
 		</joint>
-		<link name="${prefix}_linear_actuator_link">
+		<link name="${prefix}_rotary_actuator_link">
 			<inertial>
 				<origin xyz="0 0 0"/>

File: six_dof_cam_description/urdf/six_dof_cam.urdf (robot description, URDF)
Before this commit: robot six_dof_cam, 2 links, 1 joints
Links:
- removed link base_footprint
- added link map
- added link x_linear_actuator_link, mass 0.0
- added link x_rotary_actuator_link, mass 0.0
- added link y_linear_actuator_link, mass 0.0
- added link y_rotary_actuator_link, mass 0.0
- added link z_linear_actuator_link, mass 0.0
- added link z_rotary_actuator_link, mass 0.0
Joints:
- added joint x_linear_actuator_joint: type prismatic, parent map, child x_linear_actuator_link, origin xyz=0 0 0 rpy=0 0 0, axis 1 0 0, limit lower=-1 upper=1 effort=0.5 velocity=5.0
- added joint x_rotary_actuator_joint: type revolute, parent z_linear_actuator_link, child x_rotary_actuator_link, origin xyz=0 0 0 rpy=0 0 0, axis 1 0 0, limit lower=-3.14 upper=3.14 effort=0.5 velocity=5.0
- added joint y_linear_actuator_joint: type prismatic, parent x_linear_actuator_link, child y_linear_actuator_link, origin xyz=0 0 0 rpy=0 0 0, axis 0 1 0, limit lower=-1 upper=1 effort=0.5 velocity=5.0
- added joint y_rotary_actuator_joint: type revolute, parent x_rotary_actuator_link, child y_rotary_actuator_link, origin xyz=0 0 0 rpy=0 0 0, axis 0 1 0, limit lower=-3.14 upper=3.14 effort=0.5 velocity=5.0
- added joint z_linear_actuator_joint: type prismatic, parent y_linear_actuator_link, child z_linear_actuator_link, origin xyz=0 0 0 rpy=0 0 0, axis 0 0 1, limit lower=-1 upper=1 effort=0.5 velocity=5.0
- added joint z_rotary_actuator_joint: type revolute, parent y_rotary_actuator_link, child z_rotary_actuator_link, origin xyz=0 0 0 rpy=0 0 0, axis 0 0 1, limit lower=-3.14 upper=3.14 effort=0.5 velocity=5.0
- joint camera_joint: parent base_footprint -> z_rotary_actuator_link

Commit message: Fix camera description

File: six_dof_cam_description/urdf/camera/camera.xacro (robot description, xacro)
@@ -2,7 +2,5 @@
 <robot xmlns:xacro="http://ros.org/wiki/xacro">
 	<xacro:include filename="$(find six_dof_cam_description)/urdf/camera/camera.gazebo.xacro"/>
-	<!--<xacro:property name="M_PI" value="3.1415926535897931" />-->
-	<!--<xacro:property name="velocity_scale_factor" value="1.0"/>-->
-	<xacro:macro name="camera" params="parent *joint_origin">
+	<xacro:macro name="camera_model" params="parent *joint_origin">
 		<joint name="camera_joint" type="fixed">
 			<xacro:insert_block name="joint_origin"/>

File: six_dof_cam_description/urdf/six_dof_cam.xacro (robot description, xacro)
@@ -35,7 +35,7 @@
 		<axis xyz="0 0 1"/>
 	</xacro:rotary_actuator>
-	<xacro:camera parent="z_rotary_actuator_link">
+	<xacro:camera_model parent="z_rotary_actuator_link">
 		<origin xyz="0 0 0" rpy="0 0 0"/>
-	</xacro:camera>
+	</xacro:camera_model>
 <!-- ===============  Transmission =============== -->
 <xacro:linear_actuator_trans prefix="x" interface="hardware_interface/EffortJointInterface"/>
