Commit message: Gazebo上で動作するようになった

File: six_dof_cam_description/urdf/base/base.gazebo.xacro (robot description, xacro)
@@ -3,5 +3,5 @@
 	<xacro:macro name="base_gazebo">
 		<gazebo reference="base_link">
-			<!-- <selfCollide>true</selfCollide> -->
+			<!--<selfCollide>true</selfCollide>-->
 			<mu1>0.05</mu1>
 			<mu2>0.05</mu2>

File: six_dof_cam_description/urdf/camera/camera.gazebo.xacro (robot description, xacro)
@@ -3,5 +3,5 @@
 	<xacro:macro name="camera_gazebo">
 		<gazebo reference="camera_link">
-			<!-- <selfCollide>true</selfCollide> -->
+			<selfCollide>true</selfCollide>
 			<mu1>0.05</mu1>
 			<mu2>0.05</mu2>

File: six_dof_cam_description/urdf/camera/camera.xacro (robot description, xacro)
@@ -23,6 +23,6 @@
 			<inertial>
 				<origin xyz="0 0 0" rpy="0 0 0"/>
-				<mass value="1.0"/>
-				<inertia ixx="1.0" ixy="0.0" iyy="1.0" ixz="0.0" iyz="0.0" izz="1.0"/>
+				<mass value="0.01"/>
+				<inertia ixx="0.01" ixy="0.0" iyy="0.01" ixz="0.0" iyz="0.0" izz="0.01"/>
 			</inertial>
 		</link>

File: six_dof_cam_description/urdf/linear_actuator/linear_actuator.xacro (robot description, xacro)
@@ -11,5 +11,5 @@
 			<parent link="${parent}"/>
 			<child link="${prefix}_linear_actuator_link"/>
-			<limit lower="-1" upper="1" effort="0.5" velocity="5.0"/>
+			<limit lower="-1" upper="1" effort="100.0" velocity="5.0"/>
 		</joint>
 		<link name="${prefix}_linear_actuator_link">

File: six_dof_cam_description/urdf/rotary_actuator/rotary_actuator.xacro (robot description, xacro)
@@ -11,5 +11,5 @@
 			<parent link="${parent}"/>
 			<child link="${prefix}_rotary_actuator_link"/>
-			<limit lower="-3.14" upper="3.14" effort="0.5" velocity="5.0"/>
+			<limit lower="-3.14" upper="3.14" effort="5.0" velocity="5.0"/>
 		</joint>
 		<link name="${prefix}_rotary_actuator_link">
