Commit message: 6自由度できた

File: six_dof_cam_description/urdf/linear_actuator/linear_actuator.xacro (robot description, xacro)
@@ -5,10 +5,10 @@
 	<xacro:property name="velocity_scale_factor" value="1.0"/>-->
 	<xacro:macro name="linear_actuator" params="prefix parent *joint_origin *joint_axis">
-		<joint name="${prefix}_linear_actuator_joint" type="fixed">
+		<joint name="${prefix}_linear_actuator_joint" type="prismatic">
 			<insert_block name="joint_origin"/>
 			<insert_block name="joint_axis"/>
 			<parent link="${parent}"/>
 			<child link="${prefix}_linear_actuator_link"/>
-			<limit lower="-1" upper="1"/>
+			<limit lower="-1" upper="1" effort="0.5" velocity="5.0"/>
 		</joint>
 		<link name="${prefix}_linear_actuator_link">

File: six_dof_cam_description/urdf/six_dof_cam.xacro (robot description, xacro)
@@ -4,11 +4,32 @@
 	<xacro:include filename="$(find six_dof_cam_description)/urdf/camera/camera.xacro"/>
 	<xacro:include filename="$(find six_dof_cam_description)/urdf/linear_actuator/linear_actuator.xacro"/>
+	<xacro:include filename="$(find six_dof_cam_description)/urdf/rotary_actuator/rotary_actuator.xacro"/>
 <!-- =============== Link & Joint =============== -->
 	<link name="map"/>
-	<!--<xacro:linear_actuator prefix="x" parent="base_footprint">
+	<xacro:linear_actuator prefix="x" parent="map">
 		<origin xyz="0 0 0" rpy="0 0 0"/>
 		<axis xyz="1 0 0"/>
-	</xacro:linear_actuator>-->
-	<xacro:camera parent="map">
+	</xacro:linear_actuator>
+	<xacro:linear_actuator prefix="y" parent="x_linear_actuator_link">
+		<origin xyz="0 0 0" rpy="0 0 0"/>
+		<axis xyz="0 1 0"/>
+	</xacro:linear_actuator>
+	<xacro:linear_actuator prefix="z" parent="y_linear_actuator_link">
+		<origin xyz="0 0 0" rpy="0 0 0"/>
+		<axis xyz="0 0 1"/>
+	</xacro:linear_actuator>
+	<xacro:rotary_actuator prefix="x" parent="z_linear_actuator_link">
+		<origin xyz="0 0 0" rpy="0 0 0"/>
+		<axis xyz="1 0 0"/>
+	</xacro:rotary_actuator>
+	<xacro:rotary_actuator prefix="y" parent="x_rotary_actuator_link">
+		<origin xyz="0 0 0" rpy="0 0 0"/>
+		<axis xyz="0 1 0"/>
+	</xacro:rotary_actuator>
+	<xacro:rotary_actuator prefix="z" parent="y_rotary_actuator_link">
+		<origin xyz="0 0 0" rpy="0 0 0"/>
+		<axis xyz="0 0 1"/>
+	</xacro:rotary_actuator>
+	<xacro:camera parent="z_rotary_actuator_link">
 		<origin xyz="0 0 0" rpy="0 0 0"/>
 	</xacro:camera>

Commit message: fix a controller.yaml

File: six_dof_cam_description/urdf/linear_actuator/linear_actuator.xacro (robot description, xacro)
@@ -16,6 +16,6 @@
 			<inertial>
 				<origin xyz="0 0 0"/>
-				<mass value="0.0"/>
-				<inertia ixx="0.0" ixy="0.0" iyy="0.0" ixz="0.0" iyz="0.0" izz="0.0"/>
+				<mass value="1.0"/>
+				<inertia ixx="1.0" ixy="0.0" iyy="1.0" ixz="0.0" iyz="0.0" izz="1.0"/>
 			</inertial>
 		</link>

File: six_dof_cam_description/urdf/rotary_actuator/rotary_actuator.xacro (robot description, xacro)
@@ -16,6 +16,6 @@
 			<inertial>
 				<origin xyz="0 0 0"/>
-				<mass value="0.0"/>
-				<inertia ixx="0.0" ixy="0.0" iyy="0.0" ixz="0.0" iyz="0.0" izz="0.0"/>
+				<mass value="1.0"/>
+				<inertia ixx="1.0" ixy="0.0" iyy="1.0" ixz="0.0" iyz="0.0" izz="1.0"/>
 			</inertial>
 		</link>

File: six_dof_cam_description/urdf/six_dof_cam.urdf (robot description, URDF)
Before this commit: robot six_dof_cam, 8 links, 7 joints
Links:
- added link base_link, mass 1.0; collision box size=0.1 0.1 0.1; visual box size=0.1 0.1 0.1
- link x_linear_actuator_link: mass 0.0 -> 1.0
- link x_rotary_actuator_link: mass 0.0 -> 1.0
- link y_linear_actuator_link: mass 0.0 -> 1.0
- link y_rotary_actuator_link: mass 0.0 -> 1.0
- link z_linear_actuator_link: mass 0.0 -> 1.0
- link z_rotary_actuator_link: mass 0.0 -> 1.0
Joints:
- added joint base_joint: type fixed, parent world, child base_link, origin xyz=0 0 0.05 rpy=0 0 0
- joint x_linear_actuator_joint: parent world -> base_link

File: six_dof_cam_description/urdf/six_dof_cam.xacro (robot description, xacro)
@@ -3,9 +3,13 @@
 	xmlns:xacro="http://ros.org/wiki/xacro">
 	<xacro:include filename="$(find six_dof_cam_description)/urdf/camera/camera.xacro"/>
+	<xacro:include filename="$(find six_dof_cam_description)/urdf/base/base.xacro"/>
 	<xacro:include filename="$(find six_dof_cam_description)/urdf/linear_actuator/linear_actuator.xacro"/>
 	<xacro:include filename="$(find six_dof_cam_description)/urdf/rotary_actuator/rotary_actuator.xacro"/>
 <!-- =============== Link & Joint =============== -->
 	<link name="world"/>
-	<xacro:linear_actuator prefix="x" parent="world">
+	<xacro:base parent="world">
+		<origin xyz="0 0 0.05" rpy="0 0 0"/>
+	</xacro:base>
+	<xacro:linear_actuator prefix="x" parent="base_link">
 		<origin xyz="0 0 1" rpy="0 0 0"/>
 		<axis xyz="1 0 0"/>
@@ -35,10 +39,10 @@
 	</xacro:camera>
 <!-- ===============  Transmission =============== -->
-<xacro:linear_actuator_trans prefix="x" interface="hardware_interface/PositionJointInterface"/>
-<xacro:linear_actuator_trans prefix="y" interface="hardware_interface/PositionJointInterface"/>
-<xacro:linear_actuator_trans prefix="z" interface="hardware_interface/PositionJointInterface"/>
-<xacro:rotary_actuator_trans prefix="x" interface="hardware_interface/PositionJointInterface"/>
-<xacro:rotary_actuator_trans prefix="y" interface="hardware_interface/PositionJointInterface"/>
-<xacro:rotary_actuator_trans prefix="z" interface="hardware_interface/PositionJointInterface"/>
+<xacro:linear_actuator_trans prefix="x" interface="hardware_interface/EffortJointInterface"/>
+<xacro:linear_actuator_trans prefix="y" interface="hardware_interface/EffortJointInterface"/>
+<xacro:linear_actuator_trans prefix="z" interface="hardware_interface/EffortJointInterface"/>
+<xacro:rotary_actuator_trans prefix="x" interface="hardware_interface/EffortJointInterface"/>
+<xacro:rotary_actuator_trans prefix="y" interface="hardware_interface/EffortJointInterface"/>
+<xacro:rotary_actuator_trans prefix="z" interface="hardware_interface/EffortJointInterface"/>
 <!-- =============== Gazebo =============== -->
 <gazebo>
@@ -47,4 +51,6 @@
 	</plugin>
 </gazebo>
+<!-- base -->
+<xacro:base_gazebo/>
 <!-- camera -->
 <xacro:camera_gazebo/>

Commit message: Edit PID params

File: six_dof_cam_description/urdf/linear_actuator/linear_actuator.xacro (robot description, xacro)
@@ -11,5 +11,5 @@
 			<parent link="${parent}"/>
 			<child link="${prefix}_linear_actuator_link"/>
-			<limit lower="-1" upper="1" effort="100.0" velocity="5.0"/>
+			<limit lower="-3" upper="3" effort="1000.0" velocity="100.0"/>
 		</joint>
 		<link name="${prefix}_linear_actuator_link">

File: six_dof_cam_description/urdf/rotary_actuator/rotary_actuator.xacro (robot description, xacro)
@@ -11,5 +11,5 @@
 			<parent link="${parent}"/>
 			<child link="${prefix}_rotary_actuator_link"/>
-			<limit lower="-3.14" upper="3.14" effort="5.0" velocity="5.0"/>
+			<limit lower="-3.14" upper="3.14" effort="1000.0" velocity="100.0"/>
 		</joint>
 		<link name="${prefix}_rotary_actuator_link">
