Commit message: Edit base position

File: six_dof_hand_description/urdf/base/base.xacro (robot description, xacro)
@@ -15,4 +15,5 @@
 					<box size="0.1 0.1 0.1"/>
 				</geometry>
+				<origin rpy="0 0 0" xyz="-0.05 0 0.05"/>
 			</visual>
 			<collision>
@@ -20,4 +21,5 @@
 					<box size="0.1 0.1 0.1"/>
 				</geometry>
+				<origin rpy="0 0 0" xyz="-0.05 0 0.05"/>
 			</collision>
 			<inertial>

File: six_dof_hand_description/urdf/finger/finger.xacro (robot description, xacro)
@@ -17,6 +17,6 @@
 			<inertial>
 				<origin xyz="0 0 0"/>
-				<mass value="1.0"/>
-				<inertia ixx="1.0" ixy="0.0" iyy="1.0" ixz="0.0" iyz="0.0" izz="1.0"/>
+				<mass value="0.01"/>
+				<inertia ixx="0.01" ixy="0.0" iyy="0.01" ixz="0.0" iyz="0.0" izz="0.01"/>
 			</inertial>
 			<collision name="collision">
@@ -44,6 +44,6 @@
 			<inertial>
 				<origin xyz="0 0 0"/>
-				<mass value="1.0"/>
-				<inertia ixx="1.0" ixy="0.0" iyy="1.0" ixz="0.0" iyz="0.0" izz="1.0"/>
+				<mass value="0.01"/>
+				<inertia ixx="0.01" ixy="0.0" iyy="0.01" ixz="0.0" iyz="0.0" izz="0.01"/>
 			</inertial>
 			<collision name="collision">

File: six_dof_hand_description/urdf/six_dof_hand.xacro (robot description, xacro)
@@ -11,5 +11,5 @@
 	<link name="world"/>
 	<xacro:base parent="world">
-		<origin xyz="0 0 0.05" rpy="0 0 0"/>
+		<origin xyz="0 0 0" rpy="0 0 0"/>
 	</xacro:base>
 	<xacro:linear_actuator prefix="x" parent="base_link">
