Commit message: Fix direction of finger

File: six_dof_hand_description/urdf/six_dof_hand.xacro (robot description, xacro)
@@ -41,9 +41,15 @@
 	</xacro:camera_model>
 	<xacro:finger prefix="r" parent="camera_link">
+	<!--
 		<origin xyz="0.030 0.040 0" rpy="0 0 0"/>
+	-->
+		<origin xyz="0.040 -0.030 0" rpy="0 0 ${-M_PI / 2}"/>
 		<axis xyz="0 0 1"/>
 	</xacro:finger>
 	<xacro:finger prefix="l" parent="camera_link">
+	<!--
 		<origin xyz="-0.030 0.040 0" rpy="0 ${M_PI} 0"/>
+	-->
+		<origin xyz="0.040 0.030 0" rpy="0 ${M_PI} ${-M_PI / 2}"/>
 		<axis xyz="0 0 1"/>
 	</xacro:finger>

Commit message: Edit position offset

File: six_dof_hand_description/urdf/six_dof_hand.xacro (robot description, xacro)
@@ -14,5 +14,5 @@
 	</xacro:base>
 	<xacro:linear_actuator prefix="x" parent="base_link">
-		<origin xyz="0 0 1" rpy="0 0 0"/>
+		<origin xyz="0 0 0" rpy="0 0 0"/>
 		<axis xyz="1 0 0"/>
 	</xacro:linear_actuator>

Commit message: Fix finger settings

File: six_dof_hand_description/urdf/six_dof_hand.xacro (robot description, xacro)
@@ -44,5 +44,5 @@
 		<origin xyz="0.030 0.040 0" rpy="0 0 0"/>
 	-->
-		<origin xyz="0.040 -0.030 0" rpy="0 0 ${-M_PI / 2}"/>
+		<origin xyz="0.050 -0.030 0" rpy="0 0 ${-M_PI / 2}"/>
 		<axis xyz="0 0 1"/>
 	</xacro:finger>
@@ -51,5 +51,5 @@
 		<origin xyz="-0.030 0.040 0" rpy="0 ${M_PI} 0"/>
 	-->
-		<origin xyz="0.040 0.030 0" rpy="0 ${M_PI} ${-M_PI / 2}"/>
+		<origin xyz="0.050 0.030 0" rpy="0 ${M_PI} ${-M_PI / 2}"/>
 		<axis xyz="0 0 1"/>
 	</xacro:finger>
